File: hw/design/rear-light.kicad_pcb (KiCad board)
At the start: 4 copper layers, 24.6 x 64 mm, 91 parts, among them J501 Conn_ARM_SWD_TagConnect_TC203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, J705 Conn_ARM_SWD_TagConnect_TC203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, Q200 SIA469DJ-T1-GE3, SW716 KMT071 NGJ LHS, U300 MCP2003BT-E/MC, U400 TPS629210DRLR, U500 ATSAMD21E18A-M, U600 BMA456, U700 XM125, U701 AP2127N-1.8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

Commit message: Finalization (JLC ordered)
Parts:
- C808: value 2.2u -> 1u
- R712, R713, R717, R718: value 1.5k -> 1k
- R805: value 290m -> 300m
- R820: value 237k -> 200k
- R823: value 10k -> 120k
- R824: value 10k -> 27k
- R825: value 10k -> 1k
Changed lines of the file:
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@@
 			(outputformat 1)
 			(mirror no)
-			(drillshape 1)
+			(drillshape 0)
 			(scaleselection 1)
-			(outputdirectory "")
+			(outputdirectory "../../../ordering/rearlight/")
 		)
 	)
@@
 			)
 		)
-		(property "Value" "1.5k"
+		(property "Value" "1k"
 			(at -2.7 0 0)
 			(layer "B.Fab")
@@
 			)
 		)
-		(property "Value" "10k"
+		(property "Value" "120k"
 			(at -0.83 -2.32 90)
 			(layer "B.Fab")
@@
 			)
 		)
-		(property "Value" "1.5k"
+		(property "Value" "1k"
 			(at -0.02 -1.99 270)
 			(layer "B.Fab")
@@
 		(sheetname "/")
 		(sheetfile "rear-light.kicad_sch")
-		(attr smd dnp)
+		(attr smd)
 		(fp_line
 			(start -0.153641 -0.38)
@@
 			)
 		)
-		(property "Value" "1.5k"
+		(property "Value" "1k"
 			(at -2.7 0.2 0)
 			(layer "B.Fab")
@@
 			)
 		)
-		(property "Value" "237k"
+		(property "Value" "200k"
 			(at -0.7 2.2 0)
 			(layer "B.Fab")
@@
 			)
 		)
-		(property "Value" "10k"
+		(property "Value" "1k"
 			(at -0.84 -1.13 90)
 			(layer "B.Fab")
@@
 			)
 		)
-		(property "Value" "10k"
+		(property "Value" "27k"
 			(at 0.93 -2.13 90)
 			(layer "B.Fab")
@@
 		(sheetname "/")
 		(sheetfile "rear-light.kicad_sch")
-		(attr smd)
+		(attr smd dnp)
 		(fp_line
 			(start -0.261252 0.735)
@@
 		(sheetname "/")
 		(sheetfile "rear-light.kicad_sch")
-		(attr smd)
+		(attr smd dnp)
 		(fp_line
 			(start -0.107836 0.36)
@@
 			)
 		)
-		(property "Value" "290m"
+		(property "Value" "300m"
 			(at 2.5 -0.2 270)
 			(layer "B.Fab")
@@
 			)
 		)
-		(property "Value" "1.5k"
+		(property "Value" "1k"
 			(at -2.7 0.1 0)
 			(layer "B.Fab")
@@
 			)
 		)
-		(property "Value" "2.2u"
+		(property "Value" "1u"
 			(at -0.03 -1.12 0)
 			(layer "B.Fab")
