File: hw/design/rear-light.kicad_sch (KiCad schematic)
At the start: 109 parts, among them J1 Conn_ARM_SWD_TagConnect_TC203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, Q501 2N7002, Q502 2N7002, Q503 2N7002, Q601 2N7002, U300 MCP2021A-330E/SN, U400 ATSAMD21E18A-A, U500 TLD2331-3EP, U600 TLD2132-1EP, U700 BMA456

Commit message: Initial design Schematic is mostly complete
Parts:
- removed C302: 220p, Capacitor_SMD:C_0603_1608Metric, symbol Device:C
- removed C303, C304, C407, C410: 10u, Capacitor_SMD:C_0805_2012Metric, symbol Device:C
- removed C306, C408, C411, C414, C504, C602: 220n, Capacitor_SMD:C_0402_1005Metric, symbol Device:C
- removed C412: 2.2u, Capacitor_SMD:C_0805_2012Metric, symbol Device:C
- removed C509, C514, C519, C525, C607: 10n, Capacitor_SMD:C_0402_1005Metric, symbol Device:C
- removed C527, C613: 2.2n, Capacitor_SMD:C_0402_1005Metric, symbol Device:C
- removed D200: BAS3005B02, Diode_SMD:D_SOD-523, symbol Device:D_Schottky
- removed D201, D301: SMF33CA-DIO, Diode_SMD:D_SMF, symbol Device:D_TVS
- removed D506, D507, D508, D511, D512, D513, D516, D517, D518, D604, D605, D606: LED, LED_SMD:LED_0805_2012Metric, symbol Device:LED
- removed L409: 10uH, Inductor_SMD:L_0805_2012Metric, symbol Device:L
- removed Q501, Q502, Q503: 2N7002, Package_TO_SOT_SMD:SOT-23, symbol Transistor_FET:2N7002
- removed R305, R307, R413, R529, R531, R533, R536, R538, R540, R615, R619, R620, R621: 10k, Resistor_SMD:R_0402_1005Metric, symbol Device:R
- removed R403: 1k, Resistor_SMD:R_0402_1005Metric, symbol Device:R
- removed R505, R510, R515, R603: 0, Resistor_SMD:R_0603_1608Metric, symbol Device:R
- removed R520, R521, R522, R608: 18.3k, Resistor_SMD:R_0402_1005Metric, symbol Device:R
- removed R523, R609: 20k, Resistor_SMD:R_0402_1005Metric, symbol Device:R
- removed R524, R526, R528, R612, R614: 0, Resistor_SMD:R_0402_1005Metric, symbol Device:R
- removed R532: 47k, Resistor_SMD:R_0402_1005Metric, symbol Device:R
- removed R537, R539, R541, R617: 220, Resistor_SMD:R_0402_1005Metric, symbol Device:R
- removed TP1, TP10, TP11, TP12, TP13, TP14, TP15, TP16, TP2, TP20, TP21, TP22, TP23, TP3, TP4, TP5, TP6, TP7, TP8, TP9: ~, TestPoint:TestPoint_Pad_1.0x1.0mm, symbol Connector:TestPoint_Probe
- removed U100: ~, Connector_JST:JST_JWPF_B04B-JWPF-SK-R_1x04_P2.00mm_Vertical, symbol local_symbols:ECU_Connector
- removed U300: MCP2021A-330E/SN, Package_SO:SOIC-8_3.9x4.9mm_P1.27mm, symbol Interface_CAN_LIN:MCP2021A-xxxxSN
- removed U400: ATSAMD21E18A-A, Package_QFP:TQFP-32_7x7mm_P0.8mm, symbol MCU_Microchip_SAMD:ATSAMD21E18A-A
- removed U500: TLD2331-3EP, Package_SO:Infineon_PG-TSDSO-14-22, symbol local_symbols:TLD2331-3EP
- removed U600: TLD2132-1EP, Package_SO:Infineon_PG-TSDSO-14-22, symbol local_symbols:TLD2132-1EP
- added C1, C13, C15, C17, C18, C19, C6, C9: 100n, Capacitor_SMD:C_0402_1005Metric, symbol Device:C
- added C10, C22: 10u, Capacitor_SMD:C_0805_2012Metric, symbol Device:C
- added C11: 22u, Capacitor_SMD:C_0805_2012Metric, symbol Device:C
- added C12, C14, C35, C36: 10u, Capacitor_SMD:C_0402_1005Metric, symbol Device:C
- added C16: 1u, Capacitor_SMD:C_0402_1005Metric, symbol Device:C
- added C2: 100u, Capacitor_SMD:CP_Elec_6.3x5.7, symbol Device:C_Polarized_US
- added C20, C8: 100p, Capacitor_SMD:C_0402_1005Metric, symbol Device:C
- added C21: 100n, Capacitor_SMD:C_0603_1608Metric, symbol Device:C
- added C23, C24, C25, C26, C27, C28, C29, C30, C31, C32, C33, C34, C7: 10n, Capacitor_SMD:C_0402_1005Metric, symbol Device:C
- added C3: 2.2u, Capacitor_SMD:C_0805_2012Metric, symbol Device:C
- added C4: 220p, Capacitor_SMD:C_0603_1608Metric, symbol Device:C
- added C5: 22n, Capacitor_SMD:C_0603_1608Metric, symbol Device:C
- added D1 (x2): BAS3005B02, Diode_SMD:D_SOD-523, symbol Device:D_Schottky
- added D10, D11, D12, D13, D14, D15, D16, D17, D6, D7, D8, D9: LY E6SF-ABCA-36-3B5A-50, LED_SMD:LED_Cree-PLCC4_2x2mm_CW, symbol Device:LED
- added D18: XPEBRO-L1-0000-00C01, LED_SMD:LED_Cree-XP-G, symbol Device:LED
- added D2: BZT52C20-TP, Diode_SMD:D_SOD-123, symbol Device:D_Zener
- added D2: SS34F-DC, Diode_SMD:D_SMA, symbol Device:D_Schottky
- added D3: SDT23C15L02, Package_TO_SOT_SMD:SOT-23, symbol Power_Protection:SP0502BAHT
- added D5: MM5Z3V6T1G, Diode_SMD:D_SOD-523, symbol Device:D_Zener
- added J3: Conn_ARM_SWD_TagConnect_TC2030-NL, Connector:Tag-Connect_TC2030-IDC-NL_2x03_P1.27mm_Vertical, symbol Connector:Conn_ARM_SWD_TagConnect_TC2030-NL
- added J4: Conn_01x04, symbol Connector_Generic:Conn_01x04
- added L1: 22u, local:ASPI-6045, symbol Device:L
- added L2: 2.2u, Inductor_SMD:L_Coilcraft_LPS3010, symbol Device:L_Iron
- added L3: 10uH, Inductor_SMD:L_0603_1608Metric, symbol Device:L
- added Q200: SIA469DJ-T1-GE3, Package_TO_SOT_SMD:Vishay_PowerPAK_SC70-6L_Single, symbol Transistor_FET:SiA449DJ
- added R1, R16, R19, R2, R25, R4, R5, R6: 10k, Resistor_SMD:R_0402_1005Metric, symbol Device:R
- added R13, R21, R47, R7: 1k, Resistor_SMD:R_0402_1005Metric, symbol Device:R
- added R14, R3, R47 (x2): 47k, Resistor_SMD:R_0402_1005Metric, symbol Device:R
- added R15, R26, R27, R47 (x5): 4.7k, Resistor_SMD:R_0402_1005Metric, symbol Device:R
- added R18: 0, Resistor_SMD:R_0603_1608Metric, symbol Device:R
- added R20, R47: 0, Resistor_SMD:R_0402_1005Metric, symbol Device:R
- added R47: 20k, Resistor_SMD:R_0402_1005Metric, symbol Device:R
- added R8: 520m, Resistor_SMD:R_1206_3216Metric, symbol Device:R
- added TH1: ERT-J0ER103J, Resistor_SMD:R_0402_1005Metric, symbol Device:Thermistor_NTC
- added U1: ILD8150, Package_SO:Infineon_PG-DSO-8-27_3.9x4.9mm_EP2.65x3mm, symbol local:ILD8150
- added U3: TPS629210DRLR, Package_TO_SOT_SMD:SOT-583-8, symbol local_symbols:TPS629210
- added U4: ~, Connector_JST:JST_JWPF_B03B-JWPF-SK-R_1x03_P2.00mm_Vertical, symbol local_symbols:ECU_Connector
- added U5: ATSAMD21E18A-MUT, Package_DFN_QFN:VQFN-32-1EP_5x5mm_P0.5mm_EP3.5x3.5mm, symbol MCU_Microchip_SAMD:ATSAMD21E18A-A
- added U6: TLD7002-16ES, libs:SOP65P600X115-25N, symbol local_symbols:TLD7002-16ES
- added U8: XM125, libs:XM125_ACC-M, symbol XM125:XM125
- added U9: AP2127N-1.8, Package_TO_SOT_SMD:SOT-23, symbol Regulator_Linear:AP2127N-1.8
Connections:
- net +3.3V: now also C11.1, C12.2, C13.2, C35.2, D10.2 (A), D11.2 (A), D12.2 (A), D13.2 (A), D14.2 (A), D15.2 (A), D16.2 (A), D17.2 (A), D6.2 (A), D7.2 (A), D8.2 (A), D9.2 (A), J3.1 (VCC), L2.2, L3.1, R13.1, R16.1, R19.1, R20.2, R21.1, R26.1, R27.1, R47.1, R47.1, R47.1, TH1.1, U3.3 (VOS), U5.30 (VDDIN), U8.1 (VIN), U9.3 (VI)
- net +BATT: now also D3.2 (K), Q200.1 (D), U4.1
- net GND: now also C1.2, C10.1, C11.2, C12.1, C13.1, C14.1, C15.1, C16.1, C17.1, C18.1, C19.1, C2.2, C20.1, C21.2, C22.1, C23.1, C24.1, C25.1, C26.1, C27.1, C28.1, C29.1, C3.1, C30.1, C31.1, C32.1, C33.1, C34.1, C35.1, C36.1, C4.2, C6.1, C8.1, C9.1, D2.2 (A), D3.3 (A), D5.2 (A), J3.5 (GND), R15.2, R2.2, R25.1, R4.1, R47.1, R47.2, R47.2, R47.2, R6.2, R8.1, U1.4 (GND), U1.9 (EP), U3.5 (GND), U4.2, U4.5 (V_{SS}), U5.10 (GND), U5.28 (GND), U6.22 (GND), U8.10 (GND), U8.13 (GND), U8.16 (GND), U8.19 (GND), U8.2 (GND), U8.22 (GND), U8.27 (GND), U8.4 (GND), U8.7 (GND), U9.1 (GND); no longer C611.1, Q601.2 (S), R610.1, R618.1
- net M03_LINE: now also C8.2, D3.1 (K), U4.3, U4.6 (L_{BUS})
- net M03_RXD: now also R47.2, U4.1 (R_{XD}), U5.6 (PA05)
- net M03_TXD: now also U4.4 (T_{XD}), U5.5 (PA04)
- net M05_RESET: now also C17.2, J3.3 (~{RESET}), R16.2, U5.26 (~{RESET}); no longer J1.3 (~{RESET})
- net M05_SWCLK: now also J3.4 (SWCLK), R13.2, U5.31 (PA30); no longer J1.4 (SWCLK)
- net M05_SWDIO: now also J3.2 (SWDIO), U5.32 (PA31); no longer J1.2 (SWDIO)
- net VDDANA: now also C14.2, C15.2, L3.2, U5.9 (VDDANA)
- net VDDCORE: now also C16.2, U5.29 (VDDCORE)
- net VS: now also C10.2, C18.2, C2.1, C21.1, C3.2, C9.2, D2.1 (K), Q200.4 (S), R47.1, U1.8 (VIN), U3.6 (VIN), U4.7 (V_{BB}), U6.21 (VS)
- net M06_INSETa: no longer names the net of Q601.1 (G)
- net M06_INSETa: no longer R618.2
- net M07_ACCEL_INT2: no longer names the net of U700.6 (INT2)
- net TLD2132_DS: no longer names the net of C611.2
- net TLD2132_DS: no longer R610.2
- net TLD2132_INSET: no longer names the net of Q601.3 (D)
- new net: R47.2, U6.4 (VLED)
- new net: C33.2, D16.1 (K), U6.17 (OUT12)
- new net: C28.2, D11.1 (K), U6.10 (OUT5)
- new net: C32.2, D15.1 (K), U6.16 (OUT11)
- new net: C27.2, D10.1 (K), U6.9 (OUT4)
- new net: C29.2, D12.1 (K), U6.13 (OUT8)
- new net: C30.2, D13.1 (K), U6.14 (OUT9)
- new net: C31.2, D14.1 (K), U6.15 (OUT10)
- new net: C34.2, D17.1 (K), U6.18 (OUT13)
- new net: C23.2, D6.1 (K), U6.5 (OUT0)
- new net: C24.2, D7.1 (K), U6.6 (OUT1)
- new net: C25.2, D8.1 (K), U6.7 (OUT2)
- new net: C26.2, D9.1 (K), U6.8 (OUT3)
- new net: D2.2 (A), Q200.3 (G), R47.1, R47.2
- new net +1V8: C36.2, U8.3 (1V8), U9.2 (VO)
- new net ILD8150_BOOT: C5.1, D1.1 (K), U1.2 (BOOT)
- new net ILD8150_CS: C4.1, R7.1, U1.5 (CS)
- new net ILD8150_LED_N: C7.2, D18.1 (K), R7.2, R8.2
- new net ILD8150_LED_P: C7.1, D18.2 (A), L1.2, R3.2
- new net ILD8150_SW: C5.2, D2.1 (K), L1.1, U1.1 (SW)
- new net M03_EN: C19.2, U4.2 (CS), U5.4 (PA03)
- new net M03_REGEN: R14.1, U3.7 (EN), U4.8 (V_{REN})
- new net M03_VMON: D5.1 (K), R14.2, R15.1, U5.11 (PA08)
- new net M04_INPUT1_DIAG/OE: U5.7 (PA06)
- new net M04_INPUT1/~{ERR}: U5.8 (PA07)
- new net M04_INPUT2_DIAG/INPUT1: U5.12 (PA09)
- new net M04_INPUT2/INPUT2: U5.13 (PA10)
- new net M04_INPUT3_DIAG/OE: U5.14 (PA11)
- new net M04_INPUT3/~{ERR}: U5.15 (PA14)
- new net M04_NC/INPUT3: U5.16 (PA15)
- new net M04_~{SLEEP1}/DIAG1: U5.1 (PA00)
- new net M04_~{SLEEP2}/DIAG2: U5.2 (PA01)
- new net M05_BMI088_MOSI: U5.21 (PA22)
- new net M05_BMI088_SCK: U5.22 (PA23)
- new net M06_BMI088_CSA: U5.23 (PA24)
- new net M06_BMI088_CSG: U5.25 (PA27)
- new net M06_BMI088_MISO: U5.24 (PA25)
- new net M06_BMP581_CS: U5.19 (PA18)
- new net M06_BMP581_MISO: U5.20 (PA19)
- new net M06_BMP581_MOSI: U5.17 (PA16)
- new net M06_BMP581_SCK: U5.18 (PA17)
- new net M07_RADAR_BOOT: R20.1, U8.26 (MISC_GPIO2_BOOT0)
- new net M07_RADAR_DEBUG_RX: U8.21 (DEBUG_UART_RX)
- new net M07_RADAR_DEBUG_TX: U8.23 (DEBUG_UART_TX)
- new net M07_RADAR_GPIO0: U8.24 (MISC_GPIO0)
- new net M07_RADAR_GPIO1: U8.25 (MISC_GPIO1)
- new net M07_RADAR_INT: U8.28 (MCU_INT)
- new net M07_RADAR_SCL: R26.2, U8.17 (I2C_SCL)
- new net M07_RADAR_SDA: R27.2, U8.18 (I2C_SDA)
- new net M07_RADAR_SWCLK: J1.4 (SWCLK), R21.2, U8.12 (SWD_CLK)
- new net M07_RADAR_SWDIO: J1.2 (SWDIO), U8.11 (SWD_IO)
- new net M07_RADAR_WAKE: R19.2, U8.15 (WAKE_UP)
- new net M08_PWMI: R5.2, R6.1, U1.3 (DIM)
- new net M08_TEMP: R25.2, TH1.2
- new net M08_VMON: R3.1, R4.2
- new net M09_GPIO0: U6.2 (GPIN0)
- new net M09_GPIO1: U6.3 (GPIN1)
- new net M09_HSLIH: R47.1, R47.2, U6.24 (HSLIH)
- new net M09_HSLIL: C20.2, D1.2 (A), R47.2, U6.23 (HSLIL)
- new net M09_TX: D1.1 (K), R47.1
- new net TPS629210_FB: R47.1, R47.2, U3.1 (FB)
- new net TPS629210_MODE: R47.1, U3.8 (MODE)
- new net TPS629210_SW: L2.1, U3.4 (SW)
- new net VCCQ: C1.1, D1.2 (A), R1.1, R5.1, U1.7 (VCC)
- new net VDD: C22.2, R47.2, U6.1 (VDD)
- new net ~{M07_RADAR_RST}: C6.2, J1.3 (~{RESET}), U8.14 (~{RESET})
- new net ~{M08_SHUTDOWN}: R1.2, R2.1, U1.6 (~{SD})
- new net ~{M09_ERR}: U6.20 (OUT15/ERRN)
- no-connect marks 7 -> 9
Other:
- note added: "!!! VDD is 5V (10mA) !!!"
- note added: "12V / 47k = 300uA"
- note added: "3.3V / 24.7k = 133uA"
- note added: "4x ACC. SPI 2x RADAR I2C 4x RADAR UART 2x RADAR CONTROL 2x COMM UART 1x COMM CONTROL 2x INDICATOR HSLI (conflict, would need 5 SERCOM)"
- note added: "EXT. FB. AUTO PFM / PWM 2.5MHz 2.2uH"
- note added: "Keep the commutation loop small"
- note added: "Leakage 12V / 94k = 127uA"
- note added: "M02: Reverse Polarity Protection"
- note added: "M03: Communication"
- note added: "M04: DC/DC Converter"
- note added: "M05: Controller"
- note added: "M06: Accelerometer"
- note added: "M07: Radar"
- note added: "M08: Tail/Brake Light"
- note added: "M09: Turn Indicator/Hazard"
- note added: "Return path shall be clear"
- note added: "SERCOM0"
- note added: "SERCOM1"
- note added: "SERCOM3"
- note added: "TODO: RPP design minimize leakage (<10u @ 12V) minimize footprint (find different zener)"
- note added: "keep C10,C12 close to VDDIN pin of U6"
- note added: "keep C13,C15 close to VDDANA pin of U6"
- note added: "keep C17 close to VDDCORE pin of U6"
- note removed: "M02: Power conditioning M03: Communication"
- note removed: "M04: Controller"
- note removed: "M05: Tail Light"
- note removed: "M06: Brake Light"
- note removed: "M07: Accelerometer"
- note removed: "Pull-down disables outputs on POR. Series resistor limits current."
- note removed: "Pull-down disables the chip on POR. Pull-up would enable the chip by default."
- note removed: "Pull-up enables outputs on POR. (safety) Series resistor limits current."
- note removed: "Pull-up enables the chip on POR. (safety) Pull-down is not necessary for sleep condition to work."
- note removed: "Short PWMI to GND if not used."
- note removed: "When C525 is fit the channel turns off in case of a single LED short circuit."
- note removed: "When C527 is fit all the outputs turn off in case of a short/open channel."
- note removed: "When C611 is fit the channel turns off in case of a single LED short circuit."
- note removed: "When C613 is fit all the outputs turn off in case of a short/open channel."
- note removed: "keep C303 close to VBB keep C304 close to VREG"
- note removed: "keep C407,C408 close to VDDIN pin of U6"
- note removed: "keep C410,C411 close to VDDANA pin of U6"
- note removed: "keep C412 close to VDDCORE pin of U6"
- note removed: "keep C504 close to VS"
- note removed: "keep C602 close to VS"
- note removed: "keep D201,D301 close to connector"
- moved on the sheet: C611, C701, C702, FID1, FID2, FID3, FID4, Q601, R610, R618, U700

Commit message: Gen2.0 redesign - DCDC converter for LVIO - Voltage monitoring - Reverse polarity protection is P-FET - MCP2003 as LIN trans. - AL8891 LED driver - XM125 radar
Parts:
- removed C1, C18: 100n, Capacitor_SMD:C_0402_1005Metric, symbol Device:C
- removed C2: 100u, Capacitor_SMD:CP_Elec_6.3x5.7, symbol Device:C_Polarized_US
- removed C20: 100p, Capacitor_SMD:C_0402_1005Metric, symbol Device:C
- removed C21: 100n, Capacitor_SMD:C_0603_1608Metric, symbol Device:C
- removed C22: 10u, Capacitor_SMD:C_0805_2012Metric, symbol Device:C
- removed C23, C24, C25, C26, C27, C28, C29, C30, C31, C32, C33, C34, C611, C7: 10n, Capacitor_SMD:C_0402_1005Metric, symbol Device:C
- removed C3: 2.2u, Capacitor_SMD:C_0805_2012Metric, symbol Device:C
- removed C4: 220p, Capacitor_SMD:C_0603_1608Metric, symbol Device:C
- removed C5: 22n, Capacitor_SMD:C_0603_1608Metric, symbol Device:C
- removed D1 (x2): BAS3005B02, Diode_SMD:D_SOD-523, symbol Device:D_Schottky
- removed D10, D11, D12, D13, D14, D15, D16, D17, D6, D7, D8, D9: LY E6SF-ABCA-36-3B5A-50, LED_SMD:LED_Cree-PLCC4_2x2mm_CW, symbol Device:LED
- removed D18: XPEBRO-L1-0000-00C01, LED_SMD:LED_Cree-XP-G, symbol Device:LED
- removed D2: BZT52C20-TP, Diode_SMD:D_SOD-123, symbol Device:D_Zener
- removed D2: SS34F-DC, Diode_SMD:D_SMA, symbol Device:D_Schottky
- removed D3: SDT23C15L02, Package_TO_SOT_SMD:SOT-23, symbol Power_Protection:SP0502BAHT
- removed J4: Conn_01x04, symbol Connector_Generic:Conn_01x04
- removed L1: 22u, local:ASPI-6045, symbol Device:L
- removed Q601: 2N7002, Package_TO_SOT_SMD:SOT-23, symbol Transistor_FET:2N7002
- removed R18: 0, Resistor_SMD:R_0603_1608Metric, symbol Device:R
- removed R2, R25, R4, R5, R6, R618: 10k, Resistor_SMD:R_0402_1005Metric, symbol Device:R
- removed R20, R610: 0, Resistor_SMD:R_0402_1005Metric, symbol Device:R
- removed R3: 47k, Resistor_SMD:R_0402_1005Metric, symbol Device:R
- removed R47 (x3): 4.7k, Resistor_SMD:R_0402_1005Metric, symbol Device:R
- removed R47, R7: 1k, Resistor_SMD:R_0402_1005Metric, symbol Device:R
- removed R8: 520m, Resistor_SMD:R_1206_3216Metric, symbol Device:R
- removed TH1: ERT-J0ER103J, Resistor_SMD:R_0402_1005Metric, symbol Device:Thermistor_NTC
- removed U1: ILD8150, Package_SO:Infineon_PG-DSO-8-27_3.9x4.9mm_EP2.65x3mm, symbol local:ILD8150
- removed U5: ATSAMD21E18A-MUT, Package_DFN_QFN:VQFN-32-1EP_5x5mm_P0.5mm_EP3.5x3.5mm, symbol MCU_Microchip_SAMD:ATSAMD21E18A-A
- removed U6: TLD7002-16ES, libs:SOP65P600X115-25N, symbol local_symbols:TLD7002-16ES
- added C706, C806, C827, C902: 100n, Capacitor_SMD:C_0402_1005Metric, symbol Device:C
- added C801: 10u, Capacitor_SMD:C_0805_2012Metric, symbol Device:C
- added C802: 2.2u, Capacitor_SMD:C_0805_2012Metric, symbol Device:C
- added C803: 100n, Capacitor_SMD:C_0603_1608Metric, symbol Device:C
- added C808, C826: 2.2u, Capacitor_SMD:C_0402_1005Metric, symbol Device:C
- added C816: 10n, Capacitor_SMD:C_0402_1005Metric, symbol Device:C
- added D203: MM5Z20VT1G, Diode_SMD:D_SOD-523, symbol Device:D_Zener
- added D807: XPLAPR-LS-0000-00H01, LED_SMD:LED_Cree-XP, symbol Device:LED
- added L804: 22u, libs:ASPI-6045, symbol Device:L_Iron
- added R709, R812, R822, R823, R824, R825, R904: 10k, Resistor_SMD:R_0402_1005Metric, symbol Device:R
- added R712, R713, R717, R718: 1.5k, Resistor_SMD:R_0402_1005Metric, symbol Device:R
- added R805: 290m, Resistor_SMD:R_1206_3216Metric, symbol Device:R
- added R809: 150k, Resistor_SMD:R_0402_1005Metric, symbol Device:R
- added R810, R813: 100k, Resistor_SMD:R_0402_1005Metric, symbol Device:R
- added R814, R818, R819: 47k, Resistor_SMD:R_0402_1005Metric, symbol Device:R
- added R815: 200k, Resistor_SMD:R_0402_1005Metric, symbol Device:R
- added R817: 43k, Resistor_SMD:R_0402_1005Metric, symbol Device:R
- added R820: 237k, Resistor_SMD:R_0402_1005Metric, symbol Device:R
- added SW716: SW_Push, libs:KMT0, symbol Switch:SW_Push
- added TH821: ERT-J0ER103J, Resistor_SMD:R_0402_1005Metric, symbol Device:Thermistor_NTC
- added TP400, TP401, TP700, TP701, TP702: TestPoint, TestPoint:TestPoint_Pad_D1.0mm, symbol Connector:TestPoint
- added U500: ATSAMD21E18A-M, Package_DFN_QFN:QFN-32-1EP_5x5mm_P0.5mm_EP3.6x3.6mm, symbol MCU_Microchip_SAMD:ATSAMD21E18A-M
- added U800: AL8891, Package_SO:TSSOP-16-1EP_4.4x5mm_P0.65mm_EP3x3mm, symbol local_symbols:AL8891
- C602: renamed from C701; value 220n -> 100n
- C603: renamed from C702; value 220n -> 100n
- R1: value 10k -> 4.7k
- R201: renamed from R47; value 47k -> 820k
- R202: renamed from R47; value 47k -> 680k
- R704: renamed from R21; now not fitted
- R714: renamed from R26; value 4.7k -> 1.5k
- R715: renamed from R27; value 4.7k -> 1.5k
- R900: renamed from R14; value 47k -> 120k
- R901: renamed from R15; value 4.7k -> 27k
- renumbered C9 to C301, C19 to C302, C8 to C304, C10 to C401, C11 to C403, C14 to C504, C15 to C505, C12 to C506, C13 to C507, C16 to C508, C17 to C510, C35 to C702, C36 to C703, C6 to C710, D5 to D903, J3 to J501, J1 to J705, L2 to L402, L3 to L503, R47 to R303, R47 to R404, R47 to R405, R47 to R406, R13 to R502, R16 to R509, R19 to R708, U4 to U300, U3 to U400, U700 to U600, U8 to U700, U9 to U701, U4 to X100
Connections:
- net ~{M08_SHUTDOWN} is gone; now on net M03_CS: R1.2
- net +1V8: now also C706.2
- net +3.3V: now also R1.1, R709.1, R812.1, R814.1, R815.1, R818.1, SW716.2, TH821.1, TP400.1, U500.30 (VDDIN)
- net GND: now also X100.3, C706.1, C801.1, C802.1, C806.2, C808.1, C816.2, C826.1, C827.1, C902.1, D807.1 (K), R810.2, R813.2, R817.2, R819.2, R820.2, R822.1, R824.2, TP401.1, TP702.1, U500.10 (GND), U500.28 (GND), U500.33 (EP), U800.1 (PGND), U800.11 (AGND), U800.17 (EP), U800.2 (VINGND); no longer X100.2
- net M03_LINE: now also X100.2; no longer X100.3
- net M03_RXD: now also U500.12 (PA09)
- net M03_TXD: now also U500.11 (PA08)
- net M05_RESET: now also U500.26 (~{RESET})
- net M05_SWCLK: now also U500.31 (PA30)
- net M05_SWDIO: now also U500.32 (PA31)
- net M07_RADAR_BOOT: now also R717.1, U500.20 (PA19); no longer U700.26 (MISC_GPIO2_BOOT0)
- net M07_RADAR_DEBUG_RX: now also TP700.1
- net M07_RADAR_DEBUG_TX: now also TP701.1
- net M07_RADAR_GPIO0: now also R718.1, U500.27 (PA28); no longer U700.24 (MISC_GPIO0)
- net M07_RADAR_GPIO1: now also U700.24 (MISC_GPIO0); no longer U700.25 (MISC_GPIO1)
- net M07_RADAR_INT: now also U500.19 (PA18)
- net M07_RADAR_SCL: now also U500.18 (PA17)
- net M07_RADAR_SDA: now also U500.17 (PA16)
- net M07_RADAR_WAKE: now also U500.14 (PA11)
- net VCCQ: now also C808.2, U800.12 (VCC); no longer R1.1
- net VDDANA: now also U500.9 (VDDANA)
- net VDDCORE: now also U500.29 (VDDCORE)
- net VS: now also C801.2, C802.2, C827.2, D203.1 (K), R809.1, U800.3 (VIN)
- net ~{M07_RADAR_RST}: now also R709.2, U500.13 (PA10)
- net M02_RPP_GATE: now reaches Q200.3 (G), R201.2, R202.1
- net M02_RPP_GATE: now also D203.2 (A)
- net at U700.5 (UART_TX): now also R712.2
- net at U700.6 (UART_RX): now also R713.2
- net M03_EN renamed M03_CS
- net M03_CS: now also U500.8 (PA07)
- net M03_VMON renamed M07_VMON_RAW
- net M07_VMON_RAW: now also C902.2, R904.1
- net M07_ACCEL_INT1 renamed M06_INT1
- net M06_INT1: now also U500.25 (PA27)
- net M07_CS_ACCEL renamed M06_CS_ACCEL
- net M06_CS_ACCEL: now also U500.23 (PA24)
- net M07_MISO renamed M06_MISO
- net M06_MISO: now also U500.24 (PA25)
- net M07_MOSI renamed M06_MOSI
- net M06_MOSI: now also U500.21 (PA22)
- net M07_SCK renamed M06_SCK
- net M06_SCK: now also U500.22 (PA23)
- new net M07_RADAR_BOOTa: R717.2, SW716.1, U700.26 (MISC_GPIO2_BOOT0)
- new net M07_RADAR_GPIO0a: R718.2, U700.25 (MISC_GPIO1)
- new net M07_RADAR_RX: R712.1, U500.16 (PA15)
- new net M07_RADAR_TX: R713.1, U500.15 (PA14)
- new net M07_VMON: R904.2, U500.7 (PA06)
- new net M08_ADIM: C816.1, R815.2, R817.1, U500.3 (PA02), U800.7 (ADIM)
- new net M08_BOOT: C803.1, U800.15 (CBOOT)
- new net M08_CSN: C806.1, D807.2 (A), R805.1, R823.1, U800.10 (CSN)
- new net M08_CSP: L804.2, R805.2, U800.9 (CSP)
- new net M08_ENABLE: R812.2, R813.1, U500.1 (PA00), U800.4 (EN)
- new net M08_FAULT: R814.2, U500.2 (PA01), U800.13 (~{FAULT})
- new net M08_FDSET: R809.2, R810.1, U800.6 (FDSET)
- new net M08_FREQ: R820.1, U800.8 (FREQ)
- new net M08_LEDMON: C826.2, R825.1, U500.5 (PA04)
- new net M08_LEDMONa: R823.2, R824.1, R825.2
- new net M08_NTC: R822.2, TH821.2, U500.6 (PA05)
- new net M08_PDIM: R818.2, R819.1, U500.4 (PA03), U800.5 (PDIM)
- new net M08_SW: C803.2, L804.1, U800.16 (SW)
- no-connect marks 9 -> 10
Other:
- note added: "HW default ON"
- note added: "HW default ~30%"
- note added: "Keep close, guard vias"
- note added: "M06: Accelerometer/IMU"
- note added: "M09: Voltage monitoring"
- note added: "Place NTC behind LED"
- note added: "Pull down ensures off, when +3V3 is off"
- note added: "TODO: cap value"
- note added: "TODO: output capacitance?"
- note added: "TODO: resistor value"
- note added: "VCCQ=5V@30mA"
- note added: "Vinth=5V"
- note added: "keep C702 close to U700 VDDIO"
- note added: "keep C703 close to U700 VDD"
- note removed: "!!! VDD is 5V (10mA) !!!"
- note removed: "12V / 47k = 300uA"
- note removed: "Keep the commutation loop small"
- note removed: "M06: Accelerometer"
- note removed: "M09: Turn Indicator/Hazard"
- note removed: "Return path shall be clear"
- note removed: "SERCOM0"
- note removed: "SERCOM1"
- note removed: "SERCOM3"
- note removed: "keep C701 close to VDDIO"
- note removed: "keep C701,C702 close to U700"
- note removed: "keep C702 close to VDD"
- moved on the sheet: C401, C403, C510, C602, C603, C702, C703, C710, D903, FID1, FID2, FID3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

Commit message: Finalized design
Parts:
- added C828: 10u, Capacitor_SMD:C_0805_2012Metric, symbol Device:C
- R815: now fitted
- SW716: value SW_Push -> KMT071 NGJ LHS
- TP400: value TestPoint -> 3V3
- TP401, TP702: value TestPoint -> GND
- TP700: value TestPoint -> RADAR RX
- TP701: value TestPoint -> RADAR TX
- renumbered R1 to R305
Connections:
- net GND: now also C828.1
- net M08_CSN: now also C828.2
Other:
- note added: "keep C602 close to U600 VDDIO"
- note added: "keep C603 close to U600 VDD"
- note removed: "3.3V / 24.7k = 133uA"
- note removed: "4x ACC. SPI 2x RADAR I2C 4x RADAR UART 2x RADAR CONTROL 2x COMM UART 1x COMM CONTROL 2x INDICATOR HSLI (conflict, would need 5 SERCOM)"
- note removed: "TODO: output capacitance?"
- note removed: "VCCQ=5V@30mA"
- note removed: "keep C702 close to U700 VDDIO"
- note removed: "keep C703 close to U700 VDD"
- moved on the sheet: C401, C403, C504, C505, C506, C507, C508, C510, C602, C603, C702, C703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

Commit message: Finalization (JLC ordered)
Parts:
- C808: value 2.2u -> 1u
- C826, C828: now not fitted
- R305: now fitted
- R712, R713, R717, R718: value 1.5k -> 1k
- R805: value 290m -> 300m
- R820: value 237k -> 200k
- R823: value 10k -> 120k
- R824: value 10k -> 27k
- R825: value 10k -> 1k
Other:
- note removed: "TODO: cap value"
Changed lines of the file:
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@@
 		)
 	)
-	(text "TODO: resistor value"
-		(exclude_from_sim no)
-		(at 352.552 68.326 90)
-		(effects
-			(font
-				(size 1.27 1.27)
-			)
-		)
-	)
 	(text "M08: Tail/Brake Light"
 		(exclude_from_sim no)
@@
 		)
 	)
-	(text "TODO:\ncap value"
-		(exclude_from_sim no)
-		(at 265.43 52.578 0)
-		(effects
-			(font
-				(size 1.27 1.27)
-			)
-		)
-	)
 	(text "HW default ~30%"
 		(exclude_from_sim no)
@@
 		)
 	)
-	(text "TODO:\ncap value"
-		(exclude_from_sim no)
-		(at 321.31 77.47 0)
-		(effects
-			(font
-				(size 1.27 1.27)
-			)
-		)
-	)
 	(text "Vinth=5V"
 		(exclude_from_sim no)
@@
 		)
 		(property "Value" "100k"
-			(at 227.965 69.85 0)
+			(at 227.33 69.596 0)
 			(effects
 				(font
@@
 		(in_bom yes)
 		(on_board yes)
-		(dnp yes)
+		(dnp no)
 		(property "Reference" "R305"
 			(at 189.23 35.56 0)
@@
 			)
 		)
-		(property "Value" "1.5k"
+		(property "Value" "1k"
 			(at 236.22 140.97 90)
 			(effects
@@
 			)
 		)
-		(property "Value" "1.5k"
+		(property "Value" "1k"
 			(at 237.49 193.04 90)
 			(effects
@@
 			)
 		)
-		(property "Value" "10k"
+		(property "Value" "120k"
 			(at 347.345 64.77 0)
 			(effects
@@
 		(dnp no)
 		(property "Reference" "C808"
-			(at 253.365 50.8 0)
+			(at 252.73 50.8 0)
 			(effects
 				(font
@@
 			)
 		)
-		(property "Value" "2.2u"
-			(at 253.365 52.705 0)
+		(property "Value" "1u"
+			(at 254 52.578 0)
 			(effects
 				(font
@@
 		)
 		(property "Rating" "6.3V"
-			(at 253.365 54.61 0)
+			(at 252.984 54.61 0)
 			(effects
 				(font
@@
 			)
 		)
-		(property "Value" "1.5k"
+		(property "Value" "1k"
 			(at 229.87 184.15 90)
 			(effects
@@
 			)
 		)
-		(property "Value" "290m"
+		(property "Value" "300m"
 			(at 334.01 36.83 90)
 			(effects
@@
 		(in_bom yes)
 		(on_board yes)
-		(dnp no)
+		(dnp yes)
 		(property "Reference" "C828"
 			(at 346.71 43.942 0)
@@
 			)
 		)
-		(property "Value" "1.5k"
+		(property "Value" "1k"
 			(at 236.22 143.51 90)
 			(effects
@@
 			)
 		)
-		(property "Value" "10k"
+		(property "Value" "1k"
 			(at 340.36 66.04 90)
 			(effects
@@
 			)
 		)
-		(property "Value" "237k"
+		(property "Value" "200k"
 			(at 322.58 97.79 0)
 			(effects
@@
 		(in_bom yes)
 		(on_board yes)
-		(dnp no)
+		(dnp yes)
 		(property "Reference" "C826"
 			(at 326.39 72.39 0)
@@
 			)
 		)
-		(property "Value" "10k"
+		(property "Value" "27k"
 			(at 347.345 74.93 0)
 			(effects
